File: pcb/fraduino.kicad_pcb (KiCad board)
At the start: 2 copper layers, 59.8 x 96.6 mm, 82 parts, among them J1 USB_A_Board, J2 GH1.25x2, J3 SH1.0x5, Q1 SS8550, Q2 locked, Q3 SS8550, Q4 SS8550, Q5 SS8550, Q6 SS8550, Q7 SS8050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

Commit message: chg: 第一版投产
Parts:
- R22: value 0R -> 100K
- R32: value 10K -> 36K
Routing:
- net /板板/TSC_IO1: track 29.1 -> 54.4 mm, vias 2 -> 3
- net /板板/TSC_IO2: track 28.8 -> 51.8 mm, vias 2 -> 3
- net /板板/TSC_IO3: track 28.2 -> 49.7 mm, vias 2 -> 3
- added copper zone on F.Cu, net /板板/TSC_IO1
- added copper zone on F.Cu, net /板板/TSC_IO2
- added copper zone on F.Cu, net /板板/TSC_IO3
