File: pcb/fraduino.kicad_sch (KiCad schematic)
At the start: 1 part

Commit message: chg: 第一版投产
Other:
- note added: "芙兰"
Changed lines of the file:
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@@
     (comment 3 "设计: 向阳")
   )
-  (symbol (lib_id "Graphic:Logo_Open_Hardware_Large") (at 88.9 137.16 0) (unit 1)
+  (text "芙兰" (at 128.27 88.9 0)
+    (effects (font (size 8 8)) (justify left bottom))
+  )
+  (symbol (lib_id "Graphic:Logo_Open_Hardware_Large") (at 139.7 127 0) (unit 1)
     (in_bom yes) (on_board yes) (dnp no) (fields_autoplaced)
-    (property "Reference" "Sym1" (at 88.9 124.46 0)
+    (property "Reference" "Sym1" (at 139.7 114.3 0)
       (effects (font (size 1.27 1.27)) hide)
     )
-    (property "Value" "Logo_Open_Hardware_Large" (at 88.9 147.32 0)
+    (property "Value" "Logo_Open_Hardware_Large" (at 139.7 137.16 0)
       (effects (font (size 1.27 1.27)) hide)
     )
-    (property "Footprint" "Symbol:OSHW-Logo2_7.3x6mm_SilkScreen" (at 88.9 137.16 0)
+    (property "Footprint" "Symbol:OSHW-Logo2_7.3x6mm_SilkScreen" (at 139.7 127 0)
       (effects (font (size 1.27 1.27)) hide)
     )
-    (property "Datasheet" "~" (at 88.9 137.16 0)
+    (property "Datasheet" "~" (at 139.7 127 0)
       (effects (font (size 1.27 1.27)) hide)
     )
-    (property "Sim.Enable" "0" (at 88.9 137.16 0)
+    (property "Sim.Enable" "0" (at 139.7 127 0)
       (effects (font (size 1.27 1.27)) hide)
     )
@@
     )
   )
-  (sheet (at 76.2 62.23) (size 123.19 45.72) (fields_autoplaced)
+  (sheet (at 99.06 63.5) (size 83.82 36.83) (fields_autoplaced)
     (stroke (width 0.1524) (type solid))
     (fill (color 0 0 0 0.0000))
-    (property "Sheetname" "板板" (at 76.2 61.5184 0)
+    (property "Sheetname" "板板" (at 99.06 62.7884 0)
       (effects (font (size 1.27 1.27)) (justify left bottom))
     )
-    (property "Sheetfile" "main.kicad_sch" (at 76.2 108.5346 0)
+    (property "Sheetfile" "main.kicad_sch" (at 99.06 100.9146 0)
       (effects (font (size 1.27 1.27)) (justify left top))
     )
-    (property "字段 2" "" (at 76.2 62.23 0)
+    (property "字段 2" "" (at 99.06 63.5 0)
       (effects (font (size 1.27 1.27)) hide)
     )
