File: pcb/main.kicad_sch (KiCad schematic)
At the start: 81 parts, among them J1 USB_A_Board, J2 GH1.25x2, J8 SH1.0x5, Q1 SS8550, Q2 SS8550, Q3 SS8550, Q4 SS8550, Q5 SS8550, Q6 SS8550, Q7 SS8050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

Commit message: chg: 第一版投产
Parts:
- R32: value 10K -> 36K
- R42: value 0R -> 100K
Changed lines of the file:
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@@
   (title_block
     (title "Fraduino")
-    (date "2023-04-11")
+    (date "2023-06-21")
     (rev "1.0")
-    (comment 1 "审核: ")
+    (comment 1 "审核: 向阳")
     (comment 2 "制图: 向阳")
     (comment 3 "设计: 向阳")
@@
       (effects (font (size 1.27 1.27)) (justify left))
     )
-    (property "Value" "10K" (at 44.45 129.54 0)
+    (property "Value" "36K" (at 44.45 129.54 0)
       (effects (font (size 1.27 1.27)) (justify left))
     )
@@
       (effects (font (size 1.27 1.27)))
     )
-    (property "Value" "0R" (at 152.4 189.23 90)
+    (property "Value" "100K" (at 152.4 189.23 90)
       (effects (font (size 1.27 1.27)))
     )
